Commit message: ..

File: Mechanical/trial/urdf/trial (another copy).urdf (robot description, URDF)
Before this commit: robot bot, 14 links, 13 joints
Joints:
- joint EP2J: origin xyz=0 0 0.12 rpy=0 0 0 -> xyz=0 0 0 rpy=0 0 0
- joint FLWJ: origin xyz=0.125 0 0 rpy=0 0 0 -> xyz=0 0 0.12 rpy=0 0 0
- joint FRWJ: origin xyz=0.125 0 0 rpy=0 0 0 -> xyz=0 0 0.12 rpy=0 0 0
- joint RLWJ: origin xyz=-0.125 0 0 rpy=0 0 0 -> xyz=0 0 0.12 rpy=0 0 0
- joint RRWJ: origin xyz=-0.125 0 0 rpy=0 0 0 -> xyz=0 0 0.12 rpy=0 0 0
