Commit message: bot final

File: Mech2/bot1/urdf/bot1_2.urdf (robot description, URDF)
Before this commit: robot bot1, 15 links, 14 joints
Joints:
- joint BJ: axis 0 -1 0 -> 0 1 0
- joint FJ: axis 0 -1 0 -> 0 1 0
- joint FLWJ: axis 0 0 -1 -> 0 0 1
- joint LFJ: limit lower=-0.34 upper=1.36 effort=100 velocity=0.125 -> lower=-1.309 upper=0.7854 effort=100 velocity=0.125
- joint RFJ: limit lower=-1.5 upper=0.2 effort=100 velocity=0.125 -> lower=-1.309 upper=0.7854 effort=100 velocity=0.125
- joint RLWJ: axis 0 0 -1 -> 0 0 1

File: Mech2/bot1/urdf/bot1_3.urdf (robot description, URDF)
Before this commit: robot bot1, 15 links, 14 joints
Joints:
- joint LFJ: limit lower=-0.34 upper=1.36 effort=100 velocity=0.125 -> lower=-1.309 upper=0.7854 effort=100 velocity=0.125
- joint RFJ: limit lower=-1.5 upper=0.2 effort=100 velocity=0.125 -> lower=-1.309 upper=0.7854 effort=100 velocity=0.125
