Commit message: laser sensor added

File: src/mybot_description/urdf/mybot.xacro (robot description, xacro)
@@ -318,3 +318,29 @@
     </joint>
   </transmission-->
+    <joint name="hokuyo_joint" type="fixed">
+    <axis xyz="0 1 0" />
+    <origin xyz=".15 0 -.1" rpy="0 0 0"/>
+    <parent link="chassis"/>
+    <child link="hokuyo"/>
+  </joint>
+  <!-- Hokuyo Laser -->
+  <link name="hokuyo">
+    <collision>
+      <origin xyz="0 0 0" rpy="0 0 0"/>
+      <geometry>
+    <box size="0.02 0.02 0.02"/>
+      </geometry>
+    </collision>
+    <visual>
+      <origin xyz="0 0 0" rpy="0 0 0"/>
+      <geometry>
+        <box size="0.02 0.02 0.02"/>
+      </geometry>
+    </visual>
+    <inertial>
+      <mass value="1e-5" />
+      <origin xyz="0 0 0" rpy="0 0 0"/>
+      <inertia ixx="1e-6" ixy="0" ixz="0" iyy="1e-6" iyz="0" izz="1e-6" />
+    </inertial>
+  </link>
 </robot>

Commit message: Add files via upload
latest src - aryan

File: src/mybot_description/urdf/mybot.xacro (robot description, xacro)
@@ -7,5 +7,5 @@
   <xacro:include filename="$(find mybot_description)/urdf/macros.xacro" />
   <link name='chassis'>
-    <pose>0 0 0.1 0 0 0</pose>
+    <pose>0 0 0 0 0 0</pose>
     <inertial>
       <mass value="10.0"/>
@@ -21,5 +21,5 @@
         <box size=".3 .3 .2"/>
       </geometry>
-      <contact_coefficient mu="0.1"/>
+      <!--contact_coefficient mu="0.1"/-->
     </collision>
     <visual name='chassis_visual'>
@@ -245,5 +245,5 @@
   </joint-->
   <joint type="continuous" name="left_b_wheel_hinge">
-    <origin xyz="-0.12 0.1 -0.2" rpy="0 0 0"/>
+    <origin xyz="-0.12 0.1 -0.199" rpy="0 0 0"/>
     <child link="left_wheel_b"/>
     <parent link="chassis"/>
@@ -253,5 +253,5 @@
   </joint>
   <joint type="continuous" name="right_b_wheel_hinge">
-    <origin xyz="-0.12 -0.1 -0.2" rpy="0 0 0"/>
+    <origin xyz="-0.12 -0.1 -0.199" rpy="0 0 0"/>
     <child link="right_wheel_b"/>
     <parent link="chassis"/>
@@ -261,5 +261,5 @@
   </joint>
   <joint type="continuous" name="left_wheel_hinge">
-    <origin xyz="0.12 0.1 -0.2" rpy="0 0 0"/>
+    <origin xyz="0.12 0.1 -0.199" rpy="0 0 0"/>
     <child link="left_wheel"/>
     <parent link="chassis"/>
@@ -269,5 +269,5 @@
   </joint>
   <joint type="continuous" name="right_wheel_hinge">
-    <origin xyz="0.12 -0.1 -0.2" rpy="0 0 0"/>
+    <origin xyz="0.12 -0.1 -0.199" rpy="0 0 0"/>
     <child link="right_wheel"/>
     <parent link="chassis"/>
@@ -318,29 +318,3 @@
     </joint>
   </transmission-->
-    <joint name="hokuyo_joint" type="fixed">
-    <axis xyz="0 1 0" />
-    <origin xyz=".15 0 -.1" rpy="0 0 0"/>
-    <parent link="chassis"/>
-    <child link="hokuyo"/>
-  </joint>
-  <!-- Hokuyo Laser -->
-  <link name="hokuyo">
-    <collision>
-      <origin xyz="0 0 0" rpy="0 0 0"/>
-      <geometry>
-    <box size="0.02 0.02 0.02"/>
-      </geometry>
-    </collision>
-    <visual>
-      <origin xyz="0 0 0" rpy="0 0 0"/>
-      <geometry>
-        <box size="0.02 0.02 0.02"/>
-      </geometry>
-    </visual>
-    <inertial>
-      <mass value="1e-5" />
-      <origin xyz="0 0 0" rpy="0 0 0"/>
-      <inertia ixx="1e-6" ixy="0" ixz="0" iyy="1e-6" iyz="0" izz="1e-6" />
-    </inertial>
-  </link>
 </robot>
