Commit message: laser working on new bot

File: test_lidar_src/src/bot1/urdf/bot1.urdf (robot description, URDF)
Before this commit: robot bot1, 15 links, 14 joints
Links:
- removed link L
- added link hokuyo_link, mass 1e-5; collision box size=0.1 0.1 0.1; visual mesh filename=package://bot1/meshes/hokuyo.dae
Joints:
- removed joint LJ
- added joint hokuyo_joint: type fixed, parent F, child hokuyo_link, origin xyz=0.04 0.05 0 rpy=-1.57 0 0, axis 0 1 0

Commit message: added sonar for detection of dumping site

File: test_lidar_src/src/bot1/urdf/bot1.urdf (robot description, URDF)
Before this commit: robot bot1, 15 links, 14 joints
Links:
- added link sonar_link, mass 1e-5; collision box size=0.01 0.01 0.01; visual box size=0.01 0.01 0.01
Joints:
- added joint sonar_front_joint: type fixed, parent LA, child sonar_link, origin xyz=0.1 0.015 -0.02 rpy=3.1415926 0 -1.570796326, axis 0 1 0
- joint hokuyo_joint: origin xyz=0.04 0.05 0 rpy=-1.57 0 0 -> xyz=0.04 0.05 0 rpy=-1.570796326 0 0

Commit message: updates to sonar

File: test_lidar_src/src/bot1/urdf/bot1.urdf (robot description, URDF)
Before this commit: robot bot1, 16 links, 15 joints
Joints:
- joint sonar_front_joint: origin xyz=0.1 0.015 -0.02 rpy=3.1415926 0 -1.570796326 -> xyz=0.13 0.015 -0.02 rpy=3.1415926 0 -1.570796326
